File: hardware/eagle/universal-i2c-sensor-master-unit.brd (EAGLE design)
At the start: 52.1 x 74.3 mm, 35 parts, among them X1 22-23-2041, X10 22-23-2041, X11 22-23-2041, X12 22-23-2021, X13 22-23-2021, X14 22-23-2021, X2 22-23-2041, X3 22-23-2041, X4 22-23-2041, X5 22-23-2041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

Commit message: Verschönerungen
Routing:
- net SC5: track 16.0 -> 17.8 mm
- net SC4: track 18.5 -> 20.0 mm
- net SD4: track 13.4 -> 14.5 mm
- net SC6: track 14.9 -> 15.7 mm
Changed lines of the file:
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@@
 <?xml version="1.0" encoding="utf-8"?>
 <!DOCTYPE eagle SYSTEM "eagle.dtd">
-<eagle version="9.3.1">
+<eagle version="9.5.0">
 <drawing>
 <settings>
@@
 <contactref element="JP3" pad="2"/>
 <contactref element="X7" pad="3"/>
-<wire x1="33.655" y1="64.135" x2="35.56" y2="64.135" width="0.3048" layer="16"/>
-<wire x1="35.56" y1="64.135" x2="36.83" y2="65.405" width="0.3048" layer="16"/>
-<wire x1="36.83" y1="65.405" x2="41.275" y2="65.405" width="0.3048" layer="16"/>
-<wire x1="41.275" y1="65.405" x2="41.91" y2="64.77" width="0.3048" layer="16"/>
+<wire x1="41.91" y1="64.77" x2="41.275" y2="65.405" width="0.3048" layer="16"/>
 <wire x1="41.91" y1="64.77" x2="41.91" y2="62.865" width="0.3048" layer="16"/>
+<wire x1="41.275" y1="65.405" x2="38.1" y2="65.405" width="0.3048" layer="16"/>
+<wire x1="38.1" y1="65.405" x2="36.83" y2="64.135" width="0.3048" layer="16"/>
+<wire x1="36.83" y1="64.135" x2="33.655" y2="64.135" width="0.3048" layer="16"/>
 </signal>
 <signal name="SC6">
 <contactref element="JP3" pad="3"/>
 <contactref element="X6" pad="2"/>
-<wire x1="44.45" y1="55.245" x2="44.45" y2="57.785" width="0.3048" layer="16"/>
-<wire x1="43.18" y1="59.055" x2="44.45" y2="57.785" width="0.3048" layer="16"/>
-<wire x1="33.655" y1="61.595" x2="35.56" y2="61.595" width="0.3048" layer="16"/>
-<wire x1="35.56" y1="61.595" x2="38.1" y2="59.055" width="0.3048" layer="16"/>
-<wire x1="38.1" y1="59.055" x2="43.18" y2="59.055" width="0.3048" layer="16"/>
+<wire x1="36.83" y1="61.595" x2="38.1" y2="60.325" width="0.3048" layer="16"/>
+<wire x1="33.655" y1="61.595" x2="36.83" y2="61.595" width="0.3048" layer="16"/>
+<wire x1="43.18" y1="60.325" x2="44.45" y2="59.055" width="0.3048" layer="16"/>
+<wire x1="38.1" y1="60.325" x2="43.18" y2="60.325" width="0.3048" layer="16"/>
+<wire x1="44.45" y1="59.055" x2="44.45" y2="55.245" width="0.3048" layer="16"/>
 </signal>
 <signal name="SD6">
@@
 <contactref element="X6" pad="3"/>
 <wire x1="41.91" y1="55.245" x2="41.91" y2="57.15" width="0.3048" layer="16"/>
-<wire x1="41.91" y1="57.15" x2="41.275" y2="57.785" width="0.3048" layer="16"/>
-<wire x1="36.83" y1="57.785" x2="35.56" y2="59.055" width="0.3048" layer="16"/>
-<wire x1="35.56" y1="59.055" x2="33.655" y2="59.055" width="0.3048" layer="16"/>
-<wire x1="41.275" y1="57.785" x2="36.83" y2="57.785" width="0.3048" layer="16"/>
+<wire x1="41.275" y1="57.785" x2="41.91" y2="57.15" width="0.3048" layer="16"/>
+<wire x1="36.83" y1="59.055" x2="38.1" y2="57.785" width="0.3048" layer="16"/>
+<wire x1="33.655" y1="59.055" x2="36.83" y2="59.055" width="0.3048" layer="16"/>
+<wire x1="38.1" y1="57.785" x2="41.275" y2="57.785" width="0.3048" layer="16"/>
 </signal>
 <signal name="SC5">
 <contactref element="JP3" pad="5"/>
 <contactref element="X5" pad="2"/>
-<wire x1="33.655" y1="56.515" x2="35.56" y2="56.515" width="0.3048" layer="16"/>
-<wire x1="41.275" y1="52.705" x2="44.45" y2="49.53" width="0.3048" layer="16"/>
-<wire x1="44.45" y1="49.53" x2="44.45" y2="47.625" width="0.3048" layer="16"/>
-<wire x1="38.735" y1="52.705" x2="41.275" y2="52.705" width="0.3048" layer="16"/>
-<wire x1="35.56" y1="56.515" x2="36.195" y2="55.88" width="0.3048" layer="16"/>
-<wire x1="36.195" y1="55.88" x2="36.195" y2="55.245" width="0.3048" layer="16"/>
-<wire x1="36.195" y1="55.245" x2="38.735" y2="52.705" width="0.3048" layer="16"/>
+<wire x1="36.83" y1="56.515" x2="37.465" y2="55.88" width="0.3048" layer="16"/>
+<wire x1="33.655" y1="56.515" x2="36.83" y2="56.515" width="0.3048" layer="16"/>
+<wire x1="37.465" y1="55.88" x2="37.465" y2="53.975" width="0.3048" layer="16"/>
+<wire x1="43.18" y1="52.705" x2="44.45" y2="51.435" width="0.3048" layer="16"/>
+<wire x1="37.465" y1="53.975" x2="38.735" y2="52.705" width="0.3048" layer="16"/>
+<wire x1="38.735" y1="52.705" x2="43.18" y2="52.705" width="0.3048" layer="16"/>
+<wire x1="44.45" y1="51.435" x2="44.45" y2="47.625" width="0.3048" layer="16"/>
 </signal>
 <signal name="SD5">
@@
 <contactref element="X5" pad="3"/>
 <wire x1="41.91" y1="47.625" x2="41.91" y2="49.53" width="0.3048" layer="16"/>
-<wire x1="35.56" y1="53.975" x2="33.655" y2="53.975" width="0.3048" layer="16"/>
 <wire x1="41.91" y1="49.53" x2="40.005" y2="51.435" width="0.3048" layer="16"/>
-<wire x1="40.005" y1="51.435" x2="38.1" y2="51.435" width="0.3048" layer="16"/>
-<wire x1="38.1" y1="51.435" x2="35.56" y2="53.975" width="0.3048" layer="16"/>
+<wire x1="40.005" y1="51.435" x2="38.735" y2="51.435" width="0.3048" layer="16"/>
+<wire x1="38.735" y1="51.435" x2="36.195" y2="53.975" width="0.3048" layer="16"/>
+<wire x1="36.195" y1="53.975" x2="33.655" y2="53.975" width="0.3048" layer="16"/>
 </signal>
 <signal name="SC4">
 <contactref element="JP3" pad="7"/>
 <contactref element="X4" pad="2"/>
-<wire x1="33.655" y1="51.435" x2="35.56" y2="51.435" width="0.3048" layer="16"/>
-<wire x1="35.56" y1="51.435" x2="36.83" y2="50.165" width="0.3048" layer="16"/>
-<wire x1="36.83" y1="50.165" x2="39.37" y2="50.165" width="0.3048" layer="16"/>
-<wire x1="39.37" y1="50.165" x2="40.64" y2="48.895" width="0.3048" layer="16"/>
-<wire x1="44.45" y1="41.91" x2="44.45" y2="40.005" width="0.3048" layer="16"/>
-<wire x1="40.64" y1="48.895" x2="40.64" y2="45.72" width="0.3048" layer="16"/>
-<wire x1="40.64" y1="45.72" x2="44.45" y2="41.91" width="0.3048" layer="16"/>
+<wire x1="44.45" y1="43.815" x2="43.18" y2="45.085" width="0.3048" layer="16"/>
+<wire x1="43.18" y1="45.085" x2="41.275" y2="45.085" width="0.3048" layer="16"/>
+<wire x1="41.275" y1="45.085" x2="40.64" y2="45.72" width="0.3048" layer="16"/>
+<wire x1="40.64" y1="49.53" x2="40.005" y2="50.165" width="0.3048" layer="16"/>
+<wire x1="38.1" y1="50.165" x2="36.83" y2="51.435" width="0.3048" layer="16"/>
+<wire x1="44.45" y1="40.005" x2="44.45" y2="43.815" width="0.3048" layer="16"/>
+<wire x1="40.64" y1="45.72" x2="40.64" y2="49.53" width="0.3048" layer="16"/>
+<wire x1="40.005" y1="50.165" x2="38.1" y2="50.165" width="0.3048" layer="16"/>
+<wire x1="36.83" y1="51.435" x2="33.655" y2="51.435" width="0.3048" layer="16"/>
 </signal>
 <signal name="SD4">
 <contactref element="JP3" pad="8"/>
 <contactref element="X4" pad="3"/>
-<wire x1="33.655" y1="48.895" x2="35.56" y2="48.895" width="0.3048" layer="16"/>
-<wire x1="35.56" y1="48.895" x2="36.195" y2="48.26" width="0.3048" layer="16"/>
-<wire x1="36.195" y1="48.26" x2="36.195" y2="47.625" width="0.3048" layer="16"/>
-<wire x1="36.195" y1="47.625" x2="41.91" y2="41.91" width="0.3048" layer="16"/>
-<wire x1="41.91" y1="41.91" x2="41.91" y2="40.005" width="0.3048" layer="16"/>
+<wire x1="36.83" y1="48.895" x2="37.465" y2="48.26" width="0.3048" layer="16"/>
+<wire x1="37.465" y1="48.26" x2="37.465" y2="46.355" width="0.3048" layer="16"/>
+<wire x1="37.465" y1="46.355" x2="38.735" y2="45.085" width="0.3048" layer="16"/>
+<wire x1="38.735" y1="45.085" x2="39.37" y2="45.085" width="0.3048" layer="16"/>
+<wire x1="39.37" y1="45.085" x2="41.91" y2="42.545" width="0.3048" layer="16"/>
+<wire x1="33.655" y1="48.895" x2="36.83" y2="48.895" width="0.3048" layer="16"/>
+<wire x1="41.91" y1="42.545" x2="41.91" y2="40.005" width="0.3048" layer="16"/>
 </signal>
 <signal name="SC3">
